File: birdyboard.kicad_pcb (KiCad board)
At the start: 4 copper layers, 100 x 100 mm, 51 parts, among them J1 JST_3pin, J10 Conn_02x20_Odd_Even, J11 JST-PH StepMotor Conn, J12 TBP02R2-381-04BE, J13 Screw_Terminal_01x02, J14 Screw_Terminal_01x02, J15 Screw_Terminal_01x02, J16 JST-PH StepMotor Conn, J17 TBP02R2-381-04BE, J18 JST-PH StepMotor Conn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

Commit message: update component
Parts:
- U7: footprint digikey-footprints:SOT-223 -> Package_TO_SOT_SMD:SOT-89-3
- moved U7 0.13 mm to (99.4, 117.3), turned to -90 degrees
Routing:
- net +3.3V: track 65.5 -> 63.4 mm, vias 19 -> 17
